File: hardware/LOGuvnor.kicad_pcb (KiCad board)
At the start: 2 copper layers, 54 x 68.5 mm, 161 parts, among them J1 Conn_01x02, J2 Conn_01x02, J3 Conn_01x05, J4 FTDI_CONN, J5 Conn_02x04_Odd_Even, J6 Conn_01x04, J7 Si5351, J8 Conn_01x04, SW1 SW_Push_6x6, SW2 SW_Push_6x6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

Commit message: v1.2: fixes for vdd and a6/a7 pins
Parts:
- removed the G*** at (146.7, 43.8)
- removed the STCH at (149.3, 49.0)
- removed the STCH at (129.1, 33.9)
- removed the STCH at (129.1, 44.1)
- added G***: PsychoLogoMini, flyingcarsfootprints:PsychologoMini, F.Cu at (150.8, 18.4)
- added R23: R_0R_0603_JUMPER, Resistor_SMD:R_0603_1608Metric, F.Cu at (146.2, 44.4)
- added R24: R_0R_0603_JUMPER, Resistor_SMD:R_0603_1608Metric, F.Cu at (146.2, 52.2)
- added STCH: StitchingVia-0.4mmDrill, flyingcarsfootprints:StitchingVia-0.4mmDrill, F.Cu at (136.8, 32.9)
- J2: value Conn_01x02 -> Conn_02x02_Odd_Even; footprint Connector_PinSocket_2.54mm:PinSocket_1x02_P2.54mm_Vertical -> Connector_PinHeader_2.54mm:PinHeader_2x02_P2.54mm_Vertical
- moved J2 5.22 mm to (145.0, 47.0), turned to 0 degrees
- moved J1 1.48 mm to (147.3, 77.9)
- moved C1 1.10 mm to (145.5, 75.2)
- moved D3 0.40 mm to (142.5, 36.6)
- moved STCH 0.30 mm to (131.1, 31.2)
- moved D6 0.30 mm to (148.2, 36.7)
- moved STCH 0.30 mm to (155.3, 55.2)
- moved STCH 0.30 mm to (155.3, 47.3)
- moved C3 0.10 mm to (125.7, 25.9)
- moved R14 0.10 mm to (120.9, 15.0)
- moved R13 0.08 mm to (130.9, 25.9)
Connections:
- net /ROT_RAW_A renamed /Rotary_Encoder/ROT_RAW_A
- net /ROT_RAW_B renamed /Rotary_Encoder/ROT_RAW_B
- A1 pad 12: /D9 -> /CHAN_SEL_1
- A1 pad 13: /D10 -> /CHAN_EN_1
- A1 pad 25: /CHAN_SEL_1 -> unconnected-(A1-A6-Pad25)
- A1 pad 26: /CHAN_EN_1 -> unconnected-(A1-A7-Pad26)
- C10 pad 1: +3V3 -> VDD
- C7 pad 1: +3V3 -> VDD
- C8 pad 1: +3V3 -> VDD
- C9 pad 1: +3V3 -> VDD
- J2 pad 1: GND -> +3V3
- J2 pad 2: +5V -> VDD
- J3 pad 2: +3V3 -> VDD
- J4 pad 3: +3V3 -> VDD
- J5 pad 2: /D9 -> /CHAN_SEL_1
- J5 pad 5: +3V3 -> VDD
- J5 pad 8: /D10 -> /CHAN_EN_1
- J6 pad 2: +3V3 -> VDD
- J7 pad 1: +3V3 -> VDD
- J8 pad 1: +3V3 -> VDD
- R1 pad 1: +3V3 -> VDD
- R10 pad 1: +3V3 -> VDD
- R13 pad 1: +3V3 -> VDD
- R15 pad 1: +3V3 -> VDD
- R16 pad 1: +3V3 -> VDD
- R17 pad 1: +3V3 -> VDD
- R19 pad 1: +3V3 -> VDD
- R2 pad 1: +3V3 -> VDD
- R21 pad 1: +3V3 -> VDD
- R3 pad 1: +3V3 -> VDD
- R4 pad 1: +3V3 -> VDD
- R5 pad 1: +3V3 -> VDD
- R6 pad 1: +3V3 -> VDD
- R7 pad 1: +3V3 -> VDD
- R8 pad 1: +3V3 -> VDD
Routing:
- net VDD: track 0.00 -> 237.7 mm, vias 0 -> 21
- net +3V3: track 238.4 -> 57.1 mm, vias 20 -> 2
- net /CHAN_EN_1: track 33.7 -> 78.4 mm, vias 2 -> 5
- net /CHAN_SEL_1: track 31.5 -> 62.9 mm, vias 0 -> 2
- net /D10: track 14.9 -> 0.00 mm, vias 1 -> 0
- net Net-(R21-Pad2): track 6.01 -> 12.4 mm
- net Net-(R19-Pad2): track 6.01 -> 12.2 mm
- net Net-(R17-Pad2): track 6.01 -> 12.2 mm
- net /D9: track 4.51 -> 0.00 mm
- net +5V: track 4.48 -> 7.24 mm
- net /FUNC_SW: track 34.6 -> 32.4 mm
- net VAA: track 59.1 -> 60.6 mm
- net /CHAN_SEL_2: track 40.4 -> 41.0 mm
Other:
- board text added: "(C) 2023 Pat Deegan"
- board text added: "(C) 2023 Pat Deegan, psychogenic.com"
- board text added: "1EN"
- board text added: "1SL"
- board text added: "5Vin"
- board text added: "ENA"
- board text added: "Logic Level"
- board text added: "SELECT"
- board text added: "Select Switch"
- board text added: "VDD"
- board text added: "VDD Level Select"
- board text added: "v1.2"
- board text removed: "(C) 2022 Pat Deegan"
- board text removed: "(C) 2022 Pat Deegan, psychogenic.com"
- board text removed: "CHANNEL"
- board text removed: "Channel Switch"
- board text removed: "D10"
- board text removed: "D9"
- board text removed: "EN"
- board text removed: "VCC"
- board text removed: "v1.1"
