File: hardware/LOGuvnor.kicad_sch (KiCad schematic)
At the start: 37 parts, among them J1 Conn_01x02, J2 Conn_01x02, J4 FTDI_CONN, J5 Conn_02x04_Odd_Even, J6 Conn_01x04, J7 Si5351, J8 Conn_01x04

Commit message: v1.2: fixes for vdd and a6/a7 pins
Parts:
- removed J2: Conn_01x02, Connector_PinSocket_2.54mm:PinSocket_1x02_P2.54mm_Vertical, symbol Connector_Generic:Conn_01x02
- added J2: Conn_02x02_Odd_Even, Connector_PinHeader_2.54mm:PinHeader_2x02_P2.54mm_Vertical, symbol Connector_Generic:Conn_02x02_Odd_Even
- added R23, R24: R_0R_0603_JUMPER, Resistor_SMD:R_0603_1608Metric, symbol psypassives:R_0R_0603_JUMPER
Connections:
- net D10 is gone; now on net CHAN_EN_1: A1.13 (D10), J5.8 (Pin_8)
- net D9 is gone; now on net CHAN_SEL_1: A1.12 (D9), J5.2 (Pin_2)
- net +3V3: now also J2.1 (Pin_1), R23.1; no longer C10.1, C7.1, C8.1, C9.1, J4.3 (VCC), J5.5 (Pin_5), J6.2 (Pin_2), J7.1 (Pin_1), J8.1 (Pin_1), R1.1, R15.1, R16.1, R2.1, R3.1, R4.1, R5.1, R6.1, R7.1
- net +5V: now also J2.3 (Pin_3), R24.1
- net CHAN_EN_1: no longer A1.26 (A7)
- net CHAN_SEL_1: no longer A1.25 (A6)
- new net VDD: C10.1, C7.1, C8.1, C9.1, J2.2 (Pin_2), J2.4 (Pin_4), J4.3 (VCC), J5.5 (Pin_5), J6.2 (Pin_2), J7.1 (Pin_1), J8.1 (Pin_1), R1.1, R15.1, R16.1, R2.1, R23.2, R24.2, R3.1, R4.1, R5.1, R6.1, R7.1
- no-connect marks 5 -> 7
Other:
- note added: "Analog IN only"
- note added: "Logic Level Selection"
- note added: "Super simple interface to standard Si5351 modules, for ease of integration on workbench. Rotary encoder and switches, for that tactile experience. LEDs and an OLED screen for quick view of what's going on."
- note added: "populate AT MOST 1 jumper resistor"
- note added: "switchable jumper"
- note removed: "TODO:FIXME A6/A7 in only!"
- note removed: "output"
- moved on the sheet: C10, C7, C8, C9
