File: hardware/rotaryencoder.kicad_sch (KiCad schematic)
At the start: 13 parts, among them J3 Conn_01x05

Commit message: v1.2: fixes for vdd and a6/a7 pins
Connections:
- net +3V3 renamed VDD
Other:
- moved on the sheet: C5, C6, R13, R14
